Commit message: fix tf tree

File: src/turtlebot3_multi_robot/models/turtlebot3_waffle/model.sdf.xacro (robot description, xacro)
@@ -1,6 +1,8 @@
-<?xml version="1.0" ?>
-<sdf version="1.5">
-  <model name="turtlebot3_waffle">
-  <pose>0.0 0.0 0.0 0.0 0.0 0.0</pose>
+<?xml version="1.0"?>
+<sdf version="1.5" xmlns:xacro="http://www.ros.org/wiki/xacro">
+  <xacro:arg name="robot_ns" default="tb1"/>
+  <xacro:arg name="robot_name" default="turtlebot3_waffle"/>
+  <model name="$(arg robot_name)">
+    <pose>0.0 0.0 0.0 0.0 0.0 0.0</pose>
     <link name="base_footprint"/>
     <link name="base_link">
@@ -83,5 +85,5 @@
         <plugin name="turtlebot3_imu" filename="libgazebo_ros_imu_sensor.so">
           <ros>
-            <!-- <namespace>/tb3</namespace> -->
+            <namespace>/$(arg robot_ns)</namespace>
             <remapping>~/out:=imu</remapping>
           </ros>
@@ -147,5 +149,5 @@
         <plugin name="turtlebot3_laserscan" filename="libgazebo_ros_ray_sensor.so">
           <ros>
-            <!-- <namespace>/tb3</namespace> -->
+            <namespace>/$(arg robot_ns)</namespace>
             <remapping>~/out:=scan</remapping>
           </ros>
@@ -177,5 +179,4 @@
         </geometry>
         <surface>
-          <!-- This friction pamareter don't contain reliable data!! -->
           <friction>
             <ode>
@@ -231,5 +232,4 @@
         </geometry>
         <surface>
-          <!-- This friction pamareter don't contain reliable data!! -->
           <friction>
             <ode>
@@ -263,5 +263,5 @@
       </visual>
     </link>
-    <link name='caster_back_right_link'>
+    <link name="caster_back_right_link">
       <pose>-0.177 -0.064 -0.004 -1.57 0 0</pose>
       <inertial>
@@ -276,5 +276,5 @@
         </inertia>
       </inertial>
-      <collision name='collision'>
+      <collision name="collision">
         <geometry>
           <sphere>
@@ -296,5 +296,5 @@
       </collision>
     </link>
-    <link name='caster_back_left_link'>
+    <link name="caster_back_left_link">
       <pose>-0.177 0.064 -0.004 -1.57 0 0</pose>
       <inertial>
@@ -309,5 +309,5 @@
         </inertia>
       </inertial>
-      <collision name='collision'>
+      <collision name="collision">
         <geometry>
           <sphere>
@@ -345,10 +345,10 @@
       <pose>0.069 -0.047 0.107 0 0 0</pose>
       <sensor name="camera" type="depth">
-       <pose> 0 0 0 0 0 0 </pose>
+        <pose>0 0 0 0 0 0</pose>
         <always_on>true</always_on>
         <visualize>true</visualize>
         <update_rate>1</update_rate>
         <camera name="intel_realsense_r200">
-           <horizontal_fov>1.02974</horizontal_fov>
+          <horizontal_fov>1.02974</horizontal_fov>
           <image>
             <width>640</width>
@@ -357,6 +357,6 @@
           </image>
           <clip>
-               <near>0.05</near>
-               <far>8.0</far>
+            <near>0.05</near>
+            <far>8.0</far>
           </clip>
           <noise>
@@ -366,39 +366,14 @@
           </noise>
         </camera>
-          <plugin name="camera_driver" filename="libgazebo_ros_camera.so">
-            <ros>
-            </ros>
+        <plugin name="camera_driver" filename="libgazebo_ros_camera.so">
+          <ros>
+            <namespace>/$(arg robot_ns)</namespace>
+          </ros>
           <frame_name>camera_rgb_frame</frame_name>
           <min_depth>0.1</min_depth>
           <max_depth>100</max_depth>
-          </plugin>
+        </plugin>
       </sensor>
     </link>
-<!--
-  <link name="turtlebot3_wall1">
-      <visual name="turtlebot3_wall1_visual">>
-        <pose>-0.0 0 0 0 0 0</pose>
-        <geometry>
-         <box>
-            <size>0.25 0.25 0.005</size>
-         </box>
-        </geometry>
-        <material>Gazebo/Red</material>
-      </visual>
-      <collision name="turtlebot3_wall1_collision">
-        <pose>-0.0 0 .0 0 0 0</pose>
-        <geometry>
-          <box>
-            <size>0.25 0.25 0.005</size>
-         </box>
-        </geometry>
-      </collision>
-    </link>
-  <joint name="turtlebot3_wall1_joint" type="fixed">
-    <parent>turtlebot3_tray</parent>
-      <child>turtlebot3_wall1</child>
-    <pose>0.0 0.0 0.0 1.57 1.57 0</pose>
-  </joint>
-  -->
     <joint name="base_joint" type="fixed">
       <parent>base_footprint</parent>
@@ -421,9 +396,9 @@
       </axis>
     </joint>
-    <joint name='caster_back_right_joint' type='ball'>
+    <joint name="caster_back_right_joint" type="ball">
       <parent>base_link</parent>
       <child>caster_back_right_link</child>
     </joint>
-    <joint name='caster_back_left_joint' type='ball'>
+    <joint name="caster_back_left_joint" type="ball">
       <parent>base_link</parent>
       <child>caster_back_left_link</child>
@@ -463,4 +438,5 @@
     <plugin name="turtlebot3_diff_drive" filename="libgazebo_ros_diff_drive.so">
       <ros>
+        <namespace>/$(arg robot_ns)</namespace>
         <remapping>/tf:=tf</remapping>
         <remapping>/tf_static:=tf_static</remapping>
@@ -485,5 +461,5 @@
     <plugin name="turtlebot3_joint_state" filename="libgazebo_ros_joint_state_publisher.so">
       <ros>
-        <!-- <namespace>/tb3</namespace> -->
+        <namespace>/$(arg robot_ns)</namespace>
         <remapping>~/out:=joint_states</remapping>
       </ros>
