Commit message: rewrite the bringup package to work with multi robots in a real life scenario, under a single tf bus

File: src/smart_factory_bringup/models/turtlebot3_waffle/model.sdf.xacro (robot description, xacro)
@@ -5,6 +5,6 @@
   <model name="$(arg robot_name)">
     <pose>0.0 0.0 0.0 0.0 0.0 0.0</pose>
-    <link name="base_footprint"/>
-    <link name="base_link">
+    <link name="$(arg robot_ns)/base_footprint"/>
+    <link name="$(arg robot_ns)/base_link">
       <inertial>
         <pose>-0.064 0 0.048 0 0 0</pose>
@@ -37,5 +37,5 @@
       </visual>
     </link>
-    <link name="imu_link">
+    <link name="$(arg robot_ns)/imu_link">
       <sensor name="tb3_imu" type="imu">
         <always_on>true</always_on>
@@ -91,5 +91,5 @@
       </sensor>
     </link>
-    <link name="base_scan">
+    <link name="$(arg robot_ns)/base_scan">
       <inertial>
         <pose>-0.052 0 0.111 0 0 0</pose>
@@ -147,15 +147,16 @@
           </noise>
         </ray>
-        <plugin name="turtlebot3_laserscan" filename="libgazebo_ros_ray_sensor.so">
+        <plugin name="laser" filename="libgazebo_ros_ray_sensor.so">
           <ros>
             <namespace>/$(arg robot_ns)</namespace>
             <remapping>~/out:=scan</remapping>
           </ros>
+          <topic_name>scan</topic_name>
+          <frame_name>$(arg robot_ns)/base_scan</frame_name>
           <output_type>sensor_msgs/LaserScan</output_type>
-          <frame_name>base_scan</frame_name>
         </plugin>
       </sensor>
     </link>
-    <link name="wheel_left_link">
+    <link name="$(arg robot_ns)/wheel_left_link">
       <inertial>
         <pose>0.0 0.144 0.023 -1.57 0 0</pose>
@@ -210,5 +211,5 @@
       </visual>
     </link>
-    <link name="wheel_right_link">
+    <link name="$(arg robot_ns)/wheel_right_link">
       <inertial>
         <pose>0.0 -0.144 0.023 -1.57 0 0</pose>
@@ -263,5 +264,5 @@
       </visual>
     </link>
-    <link name="caster_back_right_link">
+    <link name="$(arg robot_ns)/caster_back_right_link">
       <pose>-0.177 -0.064 -0.004 -1.57 0 0</pose>
       <inertial>
@@ -296,5 +297,5 @@
       </collision>
     </link>
-    <link name="caster_back_left_link">
+    <link name="$(arg robot_ns)/caster_back_left_link">
       <pose>-0.177 0.064 -0.004 -1.57 0 0</pose>
       <inertial>
@@ -329,6 +330,6 @@
       </collision>
     </link>
-    <link name="camera_link"/>
-    <link name="camera_rgb_frame">
+    <link name="$(arg robot_ns)/camera_link"/>
+    <link name="$(arg robot_ns)/camera_rgb_frame">
       <inertial>
         <pose>0.069 -0.047 0.107 0 0 0</pose>
@@ -370,5 +371,5 @@
             <namespace>/$(arg robot_ns)</namespace>
           </ros>
-          <frame_name>camera_rgb_frame</frame_name>
+          <frame_name>$(arg robot_ns)/camera_rgb_frame</frame_name>
           <min_depth>0.1</min_depth>
           <max_depth>100</max_depth>
@@ -376,11 +377,11 @@
       </sensor>
     </link>
-    <joint name="base_joint" type="fixed">
-      <parent>base_footprint</parent>
-      <child>base_link</child>
-    </joint>
-    <joint name="wheel_left_joint" type="revolute">
-      <parent>base_link</parent>
-      <child>wheel_left_link</child>
+    <joint name="$(arg robot_ns)/base_joint" type="fixed">
+      <parent>$(arg robot_ns)/base_footprint</parent>
+      <child>$(arg robot_ns)/base_link</child>
+    </joint>
+    <joint name="$(arg robot_ns)/wheel_left_joint" type="revolute">
+      <parent>$(arg robot_ns)/base_link</parent>
+      <child>$(arg robot_ns)/wheel_left_link</child>
       <pose>0.0 0.144 0.023 -1.57 0 0</pose>
       <axis>
@@ -388,7 +389,7 @@
       </axis>
     </joint>
-    <joint name="wheel_right_joint" type="revolute">
-      <parent>base_link</parent>
-      <child>wheel_right_link</child>
+    <joint name="$(arg robot_ns)/wheel_right_joint" type="revolute">
+      <parent>$(arg robot_ns)/base_link</parent>
+      <child>$(arg robot_ns)/wheel_right_link</child>
       <pose>0.0 -0.144 0.023 -1.57 0 0</pose>
       <axis>
@@ -396,15 +397,15 @@
       </axis>
     </joint>
-    <joint name="caster_back_right_joint" type="ball">
-      <parent>base_link</parent>
-      <child>caster_back_right_link</child>
-    </joint>
-    <joint name="caster_back_left_joint" type="ball">
-      <parent>base_link</parent>
-      <child>caster_back_left_link</child>
-    </joint>
-    <joint name="imu_joint" type="fixed">
-      <parent>base_link</parent>
-      <child>imu_link</child>
+    <joint name="$(arg robot_ns)/caster_back_right_joint" type="ball">
+      <parent>$(arg robot_ns)/base_link</parent>
+      <child>$(arg robot_ns)/caster_back_right_link</child>
+    </joint>
+    <joint name="$(arg robot_ns)/caster_back_left_joint" type="ball">
+      <parent>$(arg robot_ns)/base_link</parent>
+      <child>$(arg robot_ns)/caster_back_left_link</child>
+    </joint>
+    <joint name="$(arg robot_ns)/imu_joint" type="fixed">
+      <parent>$(arg robot_ns)/base_link</parent>
+      <child>$(arg robot_ns)/imu_link</child>
       <pose>-0.032 0 0.068 0 0 0</pose>
       <axis>
@@ -412,7 +413,7 @@
       </axis>
     </joint>
-    <joint name="lidar_joint" type="fixed">
-      <parent>base_link</parent>
-      <child>base_scan</child>
+    <joint name="$(arg robot_ns)/lidar_joint" type="fixed">
+      <parent>$(arg robot_ns)/base_link</parent>
+      <child>$(arg robot_ns)/base_scan</child>
       <pose>-0.064 0 0.121 0 0 0</pose>
       <axis>
@@ -420,7 +421,7 @@
       </axis>
     </joint>
-    <joint name="camera_joint" type="fixed">
-      <parent>base_link</parent>
-      <child>camera_link</child>
+    <joint name="$(arg robot_ns)/camera_joint" type="fixed">
+      <parent>$(arg robot_ns)/base_link</parent>
+      <child>$(arg robot_ns)/camera_link</child>
       <pose>0.064 -0.065 0.094 0 0 0</pose>
       <axis>
@@ -428,7 +429,7 @@
       </axis>
     </joint>
-    <joint name="camera_rgb_joint" type="fixed">
-      <parent>camera_link</parent>
-      <child>camera_rgb_frame</child>
+    <joint name="$(arg robot_ns)/camera_rgb_joint" type="fixed">
+      <parent>$(arg robot_ns)/camera_link</parent>
+      <child>$(arg robot_ns)/camera_rgb_frame</child>
       <pose>0.005 0.018 0.013 1 0 0</pose>
       <axis>
@@ -436,15 +437,13 @@
       </axis>
     </joint>
-    <plugin name="turtlebot3_diff_drive" filename="libgazebo_ros_diff_drive.so">
+    <plugin name="diff_drive" filename="libgazebo_ros_diff_drive.so">
       <ros>
         <namespace>/$(arg robot_ns)</namespace>
-        <remapping>/tf:=tf</remapping>
-        <remapping>/tf_static:=tf_static</remapping>
         <remapping>/odom:=odom</remapping>
         <remapping>/cmd_vel:=cmd_vel</remapping>
       </ros>
       <update_rate>30</update_rate>
-      <left_joint>wheel_left_joint</left_joint>
-      <right_joint>wheel_right_joint</right_joint>
+      <left_joint>$(arg robot_ns)/wheel_left_joint</left_joint>
+      <right_joint>$(arg robot_ns)/wheel_right_joint</right_joint>
       <wheel_separation>0.287</wheel_separation>
       <wheel_diameter>0.066</wheel_diameter>
@@ -452,10 +451,10 @@
       <max_wheel_acceleration>1.0</max_wheel_acceleration>
       <command_topic>cmd_vel</command_topic>
+      <odometry_topic>odom</odometry_topic>
+      <odometry_frame>$(arg robot_ns)/odom</odometry_frame>
+      <robot_base_frame>$(arg robot_ns)/base_footprint</robot_base_frame>
       <publish_odom>true</publish_odom>
       <publish_odom_tf>true</publish_odom_tf>
       <publish_wheel_tf>false</publish_wheel_tf>
-      <odometry_topic>odom</odometry_topic>
-      <odometry_frame>odom</odometry_frame>
-      <robot_base_frame>base_footprint</robot_base_frame>
     </plugin>
     <plugin name="turtlebot3_joint_state" filename="libgazebo_ros_joint_state_publisher.so">
@@ -465,6 +464,6 @@
       </ros>
       <update_rate>30</update_rate>
-      <joint_name>wheel_left_joint</joint_name>
-      <joint_name>wheel_right_joint</joint_name>
+      <joint_name>$(arg robot_ns)/wheel_left_joint</joint_name>
+      <joint_name>$(arg robot_ns)/wheel_right_joint</joint_name>
     </plugin>
   </model>

File: src/smart_factory_bringup/urdf/turtlebot3_waffle.urdf (robot description, URDF)
Before this commit: robot turtlebot3_waffle, 13 links, 12 joints
Links:
- removed link base_footprint
- removed link base_link
- removed link base_scan
- removed link camera_depth_frame
- removed link camera_depth_optical_frame
- removed link camera_link
- removed link camera_rgb_frame
- removed link camera_rgb_optical_frame
- removed link caster_back_left_link
- removed link caster_back_right_link
- removed link imu_link
- removed link wheel_left_link
- removed link wheel_right_link
- added link ${robot_ns}/base_footprint
- added link ${robot_ns}/base_link, mass 1.3729096e+00; collision box size=0.266 0.266 0.094; visual mesh filename=package://turtlebot3_gazebo/models/turtlebot3_common/meshes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 scale=0.001 0.001 0.001
- added link ${robot_ns}/base_scan, mass 0.114; collision cylinder length=0.0315 radius=0.055; visual mesh filename=package://turtlebot3_gazebo/models/turtlebot3_common/meshes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 scale=0.001 0.001 0.001
- added link ${robot_ns}/camera_depth_frame
- added link ${robot_ns}/camera_depth_optical_frame
- added link ${robot_ns}/camera_link; collision box size=0.012 0.132 0.020; visual mesh filename=package://turtlebot3_gazebo/models/turtlebot3_common/meshes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
- added link ${robot_ns}/camera_rgb_frame
- added link ${robot_ns}/camera_rgb_optical_frame
- added link ${robot_ns}/caster_back_left_link, mass 0.005; collision box size=0.030 0.009 0.020
- added link ${robot_ns}/caster_back_right_link, mass 0.005; collision box size=0.030 0.009 0.020
- added link ${robot_ns}/imu_link
- added link ${robot_ns}/wheel_left_link, mass 2.8498940e-02; collision cylinder length=0.018 radius=0.033; visual mesh filename=package://turtlebot3_gazebo/models/turtlebot3_common/meshes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 scale=0.001 0.001 0.001
- added link ${robot_ns}/wheel_right_link, mass 2.8498940e-02; collision cylinder length=0.018 radius=0.033; visual mesh filename=package://turtlebot3_gazebo/models/turtlebot3_common/meshes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 scale=0.001 0.001 0.001
Joints:
- removed joint base_joint
- removed joint camera_depth_joint
- removed joint camera_depth_optical_joint
- removed joint camera_joint
- removed joint camera_rgb_joint
- removed joint camera_rgb_optical_joint
- removed joint caster_back_left_joint
- removed joint caster_back_right_joint
- removed joint imu_joint
- removed joint scan_joint
- removed joint wheel_left_joint
- removed joint wheel_right_joint
- added joint ${robot_ns}/base_joint: type fixed, parent ${robot_ns}/base_footprint, child ${robot_ns}/base_link, origin xyz=0 0 0.010 rpy=0 0 0
- added joint ${robot_ns}/camera_depth_joint: type fixed, parent ${robot_ns}/camera_link, child ${robot_ns}/camera_depth_frame, origin xyz=0.005 0.028 0.013 rpy=0 0 0
- added joint ${robot_ns}/camera_depth_optical_joint: type fixed, parent ${robot_ns}/camera_depth_frame, child ${robot_ns}/camera_depth_optical_frame, origin xyz=0 0 0 rpy=-1.57 0 -1.57
- added joint ${robot_ns}/camera_joint: type fixed, parent ${robot_ns}/base_link, child ${robot_ns}/camera_link, origin xyz=0.064 -0.065 0.094 rpy=0 0 0
- added joint ${robot_ns}/camera_rgb_joint: type fixed, parent ${robot_ns}/camera_link, child ${robot_ns}/camera_rgb_frame, origin xyz=0.005 0.018 0.013 rpy=0 0 0
- added joint ${robot_ns}/camera_rgb_optical_joint: type fixed, parent ${robot_ns}/camera_rgb_frame, child ${robot_ns}/camera_rgb_optical_frame, origin xyz=0 0 0 rpy=-1.57 0 -1.57
- added joint ${robot_ns}/caster_back_left_joint: type fixed, parent ${robot_ns}/base_link, child ${robot_ns}/caster_back_left_link, origin xyz=-0.177 0.064 -0.004 rpy=-1.57 0 0
- added joint ${robot_ns}/caster_back_right_joint: type fixed, parent ${robot_ns}/base_link, child ${robot_ns}/caster_back_right_link, origin xyz=-0.177 -0.064 -0.004 rpy=-1.57 0 0
- added joint ${robot_ns}/imu_joint: type fixed, parent ${robot_ns}/base_link, child ${robot_ns}/imu_link, origin xyz=0.0 0 0.068 rpy=0 0 0
- added joint ${robot_ns}/scan_joint: type fixed, parent ${robot_ns}/base_link, child ${robot_ns}/base_scan, origin xyz=-0.064 0 0.122 rpy=0 0 0
- added joint ${robot_ns}/wheel_left_joint: type continuous, parent ${robot_ns}/base_link, child ${robot_ns}/wheel_left_link, origin xyz=0.0 0.144 0.023 rpy=-1.57 0 0, axis 0 0 1
- added joint ${robot_ns}/wheel_right_joint: type continuous, parent ${robot_ns}/base_link, child ${robot_ns}/wheel_right_link, origin xyz=0.0 -0.144 0.023 rpy=-1.57 0 0, axis 0 0 1
